File: ah3000.kicad_pcb (KiCad board)
At the start: 2 copper layers, 163.8 x 95.8 mm, 116 parts, among them IC1 L487, IC2 Conn_02x20_Counter_Clockwise, IC3 CA3130, IC4 4051, IC5 M74HC4066B1R, SW0 SW_7WAY, SW1 SW_Push_AH, SW2 SW_Push_AH, SW3 SW_Push_AH, SW4 SW_Push_AH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

Commit message: Set paper size to A3, and adjusted schematic to fit.  Added PDF.
Connections:
- R32 pad 1: Net-(R32-Pad1) -> +12V
- R32 pad 2: +12V -> Net-(R32-Pad2)
- TR12 pad 1: Net-(R32-Pad1) -> Net-(R32-Pad2)
- TR8 pad 1: Net-(R32-Pad1) -> Net-(R32-Pad2)
- TR9 pad 3: Net-(R32-Pad1) -> Net-(R32-Pad2)
